File: interface-2-cart-bugged-romcs/interface-2-cart.sch (EAGLE design)
At the start: 51 parts, among them U1 SN74LVC245ADBR, U3 W25Q128JVSIQ, U4 SN74LVC245ADBR, U5 SN74LVC245ADBR, X2 TSX-32250, X3 DNP

Commit message: New version of IF2 cart, fixed bug
Parts:
- removed R1, R2, R3, R4, R5, R6, R7, R8: 10K, res-small-footprint:RES-0402
- removed U1: SN74LVC245ADBR, SN74LVC245ADBR:SN74LVC245ADBR
- added C12: 1uF, res-small-footprint:CAP-0402
- added U6: SN74LVCC4245APWR, SN74LVCC4245APWR:SN74LVCC4245APWR
- C1, C10: value 4u7 -> 100nF
- C23: value 4u7 -> 2u2
- C24: value 100nF -> 2u2
- C28: value 4u7 -> 10uF
- renumbered C6 to C10
Connections:
- net /ROMCS_3V3: now also U6.DIR; no longer U1.DIR
- net 3V3: now also C12.2, U6.VCCB
- net D0: now also U6.B1; no longer R8.2, U1.A8
- net D0_5V: now also U6.A1; no longer U1.B8
- net D1: now also U6.B2; no longer R7.2, U1.A7
- net D1_5V: now also U6.A2; no longer U1.B7
- net D2: now also U6.B3; no longer R6.2, U1.A6
- net D2_5V: now also U6.A3; no longer U1.B6
- net D3: now also U6.B4; no longer R5.2, U1.A5
- net D3_5V: now also U6.A4; no longer U1.B5
- net D4: now also U6.B5; no longer R4.2, U1.A4
- net D4_5V: now also U6.A5; no longer U1.B4
- net D5: now also U6.B6; no longer R3.2, U1.A3
- net D5_5V: now also U6.A6; no longer U1.B3
- net D6: now also U6.B7; no longer R2.2, U1.A2
- net D6_5V: now also U6.A7; no longer U1.B2
- net D7: now also U6.B8; no longer R1.2, U1.A1
- net D7_5V: now also U6.A8; no longer U1.B1
- net GND: now also C12.1, U6.GND, U6.GND-1, U6.GND-2; no longer R1.1, R2.1, R3.1, R4.1, R5.1, R6.1, R7.1, R8.1, U1.GND
- net ROMRQ_3V3: now also U6./OE; no longer U1.~OE
- net VCC: now also U6.VCCA; no longer U1.VCC
Other:
- moved on the sheet: C2, C4
