File: interface-2-cart/interface-2-cart.sch (EAGLE design)
At the start: 51 parts, among them U1 SN74LVC245ADBR, U3 W25Q128JVSIQ, U4 SN74LVC245ADBR, U5 SN74LVC245ADBR, X2 TSX-32250, X3 DNP

Commit message: Finished redesign of IF2 PCB - all data and address tracks now length matched, although whether that makes any difference... Submitted for production
Parts:
- removed S_LED10: 20mA, led-0402:VLMW1500-GS08
- added ACT_LED: 20mA, 52101-101-REV-A_v16:LED_LEDCHIP-LED0603MP
- added USER_BUTTON: PTS645SM43SMTR92LFS, PTS645SM43SMTR92LFS:PTS645SM43SMTR92LFS
- 3V3_REG2: value 3V3 -> MCP1703CB; device IC-packages_BIG-pack V1.0:NCP718BSN330T1G -> linear:MCP1703CB
Connections:
- new net USER_BUT: USER_BUTTON.3, X3.GPIO28/AD2
- net 3V3: now also 3V3_REG2.VO; no longer 3V3_REG2.OUT
- net GND: now also ACT_LED.C, USER_BUTTON.1; no longer S_LED10.C
- net N$6: now also ACT_LED.A; no longer S_LED10.A
- net VCC: now also 3V3_REG2.VI; no longer 3V3_REG2.EN, 3V3_REG2.IN
Other:
- note added: "Flash Memory"
- note added: "Interface Logic"
- note added: "Microcontroller"
- note added: "Ports"
- note added: "Power Supply"
- note added: "UI"
- moved on the sheet: C1, C11, C13, C14, C15, C16, C17, C18, C19, C2, C20, C21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

Commit message: Final(?) design of IF2 PCB.
Parts:
- removed U4, U5: SN74LVC245ADBR, SN74LVC245ADBR:SN74LVC245ADBR
- added U0, U2: SOP65P640X110-20N, SOP65P640X110-20N:SOP65P640X110-20N
- D2, D3: value BZX384C5V6-E3-08 -> (none); device BZX384C5V6-E3-08:BZX384C5V6-E3-08 -> adafruit:DIODESOD-323F
- U1: value SN74LVC245ADBR -> SOP65P640X110-20N; device SN74LVC245ADBR:SN74LVC245ADBR -> SOP65P640X110-20N:SOP65P640X110-20N
Connections:
- net /RESET_3V3: now also U2.B1; no longer U5.B2
- net /ROMCS_3V3: now also U0.DIR; no longer U1.DIR
- net 3V3: now also U1.VCC, U2.VCC; no longer U4.VCC, U5.VCC
- net A0: now also U1.A7; no longer U4.A8
- net A0_5V: now also U1.B7; no longer U4.B8
- net A1: now also U1.A6; no longer U4.A7
- net A10: now also U2.A5; no longer U5.A6
- net A10_5V: now also U2.B5; no longer U5.B6
- net A11: now also U2.A4; no longer U5.A5
- net A11_5V: now also U2.B4; no longer U5.B5
- net A12: now also U2.A3; no longer U5.A4
- net A12_5V: now also U2.B3; no longer U5.B4
- net A13: now also U2.A2; no longer U5.A3
- net A13_5V: now also U2.B2; no longer U5.B3
- net A1_5V: now also U1.B6; no longer U4.B7
- net A2: now also U1.A5; no longer U4.A6
- net A2_5V: now also U1.B5; no longer U4.B6
- net A3: now also U1.A4; no longer U4.A5
- net A3_5V: now also U1.B4; no longer U4.B5
- net A4: now also U1.A3; no longer U4.A4
- net A4_5V: now also U1.B3; no longer U4.B4
- net A5: now also U1.A2; no longer U4.A3
- net A5_5V: now also U1.B2; no longer U4.B3
- net A6: now also U1.A1; no longer U4.A2
- net A6_5V: now also U1.B1; no longer U4.B2
- net A7: now also U1.A0; no longer U4.A1
- net A7_5V: now also U1.B0; no longer U4.B1
- net A8: now also U2.A7; no longer U5.A8
- net A8_5V: now also U2.B7; no longer U5.B8
- net A9: now also U2.A6; no longer U5.A7
- net A9_5V: now also U2.B6; no longer U5.B7
- net D0: now also U0.A7; no longer U1.A8
- net D0_5V: now also U0.B7; no longer U1.B8
- net D1: now also U0.A6; no longer U1.A7
- net D1_5V: now also U0.B6; no longer U1.B7
- net D2: now also U0.A5; no longer U1.A6
- net D2_5V: now also U0.B5; no longer U1.B6
- net D3: now also U0.A4; no longer U1.A5
- net D3_5V: now also U0.B4; no longer U1.B5
- net D4: now also U0.A3; no longer U1.A4
- net D4_5V: now also U0.B3; no longer U1.B4
- net D5: now also U0.A2; no longer U1.A3
- net D5_5V: now also U0.B2; no longer U1.B3
- net D6: now also U0.A1; no longer U1.A2
- net D6_5V: now also U0.B1; no longer U1.B2
- net D7: now also U0.A0; no longer U1.A1
- net D7_5V: now also U0.B0; no longer U1.B1
- net GND: now also U0.GND, U1./OE, U1.DIR, U2./OE, U2.DIR, U2.GND; no longer U4.DIR, U4.GND, U4.~OE, U5.DIR, U5.GND, U5.~OE
- net N$9: now also U2.A1; no longer U5.A2
- net ROMRQ: now also U2.B0; no longer U5.B1
- net ROMRQ_3V3: now also U0./OE, U2.A0; no longer U1.~OE, U5.A1
- net VCC: now also U0.VCC; no longer U1.VCC
Other:
- moved on the sheet: C2, C23, C24, C3, C4, R25, R9
