File: interface-2-cart/interface-2-cart.brd (EAGLE design)
At the start: 38.7 x 35.8 mm, 52 parts, among them U0 SOP65P640X110-20N, U1 SOP65P640X110-20N, U2 SOP65P640X110-20N, U3 W25Q128JVSIQ, X2 TSX-32250, X3 DNP

Commit message: New emulator code
Routing:
- net A0_5V: track 9.16 -> 26.8 mm
- net A9_5V: track 10.4 -> 26.8 mm
- net A1_5V: track 10.5 -> 26.7 mm
- net /MREQ: track 13.1 -> 26.8 mm
- net A3_5V: track 14.1 -> 26.8 mm
- net A11_5V: track 14.7 -> 26.8 mm
- net A4_5V: track 15.6 -> 26.8 mm, vias 1 -> 2
- net A10_5V: track 15.6 -> 26.8 mm
- net A2_5V: track 15.8 -> 26.8 mm
- net A14_5V: track 16.8 -> 26.8 mm
- net A8_5V: track 18.4 -> 26.8 mm
- net A12_5V: track 18.5 -> 26.8 mm
- net A13_5V: track 19.0 -> 26.8 mm
- net D4_5V: track 8.46 -> 15.2 mm
- net D2_5V: track 8.57 -> 15.2 mm
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